Commit message: gazebo-classic

File: src/my_robot_description/urdf/arm.xacro (robot description, xacro)
@@ -22,6 +22,6 @@
             <origin xyz="0 0 ${arm_base_height / 2.0}" rpy="0 0 0" />
         </collision>
-        <xacro:box_inertia m="0.5" x="${arm_base_length}" y="${arm_base_width}" z="${arm_base_height}"
-                           o_xyz="0 0 ${arm_base_height / 2.0}" o_rpy="0 0 0" />
+        <xacro:box_inertia m="0.5" l="${2*arm_base_length}" w="${2*arm_base_width}" h="${2*arm_base_height}"
+                           xyz="0 0 ${arm_base_height / 2.0}" rpy="0 0 0" />
     </link>
     <link name="forearm_link">
@@ -39,6 +39,6 @@
             <origin xyz="0 0 ${forearm_length / 2.0}" rpy="0 0 0" />
         </collision>
-        <xacro:cylinder_inertia m="0.3" r="${forearm_radius}" l="${forearm_length}"
-                                o_xyz="0 0 ${forearm_length / 2.0}" o_rpy="0 0 0" />
+        <xacro:cylinder_inertia m="0.3" r="${2*forearm_radius}" h="${2*forearm_length}"
+                                xyz="0 0 ${forearm_length / 2.0}" rpy="0 0 0" />
     </link>
     <link name="hand_link">
@@ -51,11 +51,11 @@
         </visual>
         <collision>
-            <geometry>
+             <geometry>
                 <cylinder radius="${hand_radius}" length="${hand_length}" />
             </geometry>
             <origin xyz="0 0 ${hand_length / 2.0}" rpy="0 0 0" />
         </collision>
-        <xacro:cylinder_inertia m="0.3" r="${hand_radius}" l="${hand_length}"
-                                o_xyz="0 0 ${hand_length / 2.0}" o_rpy="0 0 0" />
+        <xacro:cylinder_inertia m="0.3" r="${2*hand_radius}" h="${2*hand_length}"
+                                xyz="0 0 ${hand_length / 2.0}" rpy="0 0 0" />
     </link>
     <joint name="arm_base_forearm_joint" type="revolute">
@@ -65,5 +65,5 @@
         <axis xyz="0 1 0" />
         <limit lower="0" upper="${pi/2}" effort="100" velocity="100" />
-        <dynamics friction="0.3" damping="0.3" />
+        <dynamics friction="0.05" damping="0.1" />
     </joint>
     <joint name="forearm_hand_joint" type="revolute">
@@ -73,5 +73,5 @@
         <axis xyz="0 1 0" />
         <limit lower="0" upper="${pi/2}" effort="100" velocity="100" />
-        <dynamics friction="0.3" damping="0.3" />
+        <dynamics friction="0.05" damping="0.1" />
     </joint>
 </robot>

File: src/my_robot_description/urdf/arm_gazebo.xacro (robot description, xacro)
@@ -1,27 +1,29 @@
 <?xml version="1.0"?>
 <robot xmlns:xacro="http://www.ros.org/wiki/xacro">
-    <gazebo>
-        <plugin
-            filename="gz-sim-joint-position-controller-system"
-            name="gz::sim::systems::JointPositionController">
-            <joint_name>arm_base_forearm_joint</joint_name>
-            <p_gain>5.0</p_gain>
-        </plugin>
+    <gazebo reference="arm_base_link">
+        <material>Gazebo/Orange</material>
+    </gazebo>
+    <gazebo reference="forearm_link">
+        <material>Gazebo/Yellow</material>
+    </gazebo>
+    <gazebo reference="hand_link">
+        <material>Gazebo/Orange</material>
     </gazebo>
     <gazebo>
-        <plugin
-            filename="gz-sim-joint-position-controller-system"
-            name="gz::sim::systems::JointPositionController">
-            <joint_name>forearm_hand_joint</joint_name>
-            <p_gain>3.0</p_gain>
-        </plugin>
-    </gazebo>
-    <gazebo>
-        <plugin
-            filename="gz-sim-joint-state-publisher-system"
-            name="gz::sim::systems::JointStatePublisher">
+        <plugin name="joint_state_publisher_controller"
+                filename="libgazebo_ros_joint_state_publisher.so">
+            <!-- Update rate in Hertz -->
+            <update_rate>10</update_rate>
+            <!-- Name of joints in the model whose states will be published. -->
             <joint_name>arm_base_forearm_joint</joint_name>
             <joint_name>forearm_hand_joint</joint_name>
         </plugin>
     </gazebo>
+    <gazebo>
+        <plugin name="joint_pose_trajectory_controller"
+                filename="libgazebo_ros_joint_pose_trajectory.so">
+            <!-- Update rate in Hz -->
+            <update_rate>2</update_rate>
+        </plugin>
+    </gazebo>
 </robot>

File: src/my_robot_description/urdf/camera.xacro (robot description, xacro)
@@ -16,6 +16,6 @@
             </geometry>
         </collision>
-        <xacro:box_inertia m="0.1" x="${camera_length}" y="${camera_width}" z="${camera_height}"
-                           o_xyz="0 0 0" o_rpy="0 0 0" />
+        <xacro:box_inertia m="0.1" l="${camera_length}" w="${camera_width}" h="${camera_height}"
+                           xyz="0 0 0" rpy="0 0 0" />
     </link>
     <joint name="base_camera_joint" type="fixed">
@@ -24,6 +24,10 @@
         <origin xyz="${(base_length + camera_length) / 2.0} 0 ${base_height / 2.0}" rpy="0 0 0" />
     </joint>
-    <link name="camera_link_optical" />
+    <link name="camera_link_optical">
+    </link>
     <joint name="camera_optical_joint" type="fixed">
+        <!-- these values have to be these values otherwise the gazebo camera
+            image won't be aligned properly with the frame it is supposedly
+            originating from -->
         <origin xyz="0 0 0" rpy="${-pi/2} 0 ${-pi/2}"/>
         <parent link="camera_link"/>
@@ -31,28 +35,12 @@
     </joint>
     <gazebo reference="camera_link">
-        <sensor name="camera" type="camera">
-            <camera>
-                <horizontal_fov>1.3962634</horizontal_fov>
-                <image>
-                    <width>640</width>
-                    <height>480</height>
-                    <format>R8G8B8</format>
-                </image>
-                <clip>
-                    <near>0.1</near>
-                    <far>15</far>
-                </clip>
-                <noise>
-                    <type>gaussian</type>
-                    <mean>0.0</mean>
-                    <stddev>0.007</stddev>
-                </noise>
-                <optical_frame_id>camera_link_optical</optical_frame_id>
-                <camera_info_topic>camera/camera_info</camera_info_topic>
-            </camera>
-            <always_on>1</always_on>
-            <update_rate>20</update_rate>
+        <material>Gazebo/Red</material>
+        <sensor name="camera_sensor" type="camera">
+            <pose>0 0 0 0 0 0</pose>
             <visualize>true</visualize>
-            <topic>camera/image_raw</topic>
+            <update_rate>10.0</update_rate>
+            <plugin name="camera_controller" filename="libgazebo_ros_camera.so">
+                <frame_name>camera_link_optical</frame_name>
+            </plugin>
         </sensor>
     </gazebo>

File: src/my_robot_description/urdf/common_properties.xacro (robot description, xacro)
@@ -13,26 +13,26 @@
         <color rgba="1.0 1.0 0 1" />
     </material>
-    <xacro:macro name="box_inertia" params="m x y z o_xyz o_rpy">
+    <xacro:macro name="box_inertia" params="m l w h xyz rpy">
         <inertial>
+            <origin xyz="${xyz}" rpy="${rpy}" />
             <mass value="${m}" />
-            <origin xyz="${o_xyz}" rpy="${o_rpy}" />
-            <inertia ixx="${(m/12) * (y*y + z*z)}" ixy="0" ixz="0"
-                     iyy="${(m/12) * (x*x + z*z)}" iyz="0"
-                     izz="${(m/12) * (x*x + y*y)}" />
+            <inertia ixx="${(m/12) * (h*h + l*l)}" ixy="0" ixz="0"
+                     iyy="${(m/12) * (w*w + l*l)}" iyz="0"
+                     izz="${(m/12) * (w*w + h*h)}" />
         </inertial>
     </xacro:macro>
-    <xacro:macro name="cylinder_inertia" params="m r l o_xyz o_rpy">
+    <xacro:macro name="cylinder_inertia" params="m r h xyz rpy">
         <inertial>
+            <origin xyz="${xyz}" rpy="${rpy}" />
             <mass value="${m}" />
-            <origin xyz="${o_xyz}" rpy="${o_rpy}" />
-            <inertia ixx="${(m/12) * (3*r*r + l*l)}" ixy="0" ixz="0"
-                     iyy="${(m/12) * (3*r*r + l*l)}" iyz="0"
+            <inertia ixx="${(m/12) * (3*r*r + h*h)}" ixy="0" ixz="0"
+                     iyy="${(m/12) * (3*r*r + h*h)}" iyz="0"
                      izz="${(m/2) * (r*r)}" />
         </inertial>
     </xacro:macro>
-    <xacro:macro name="sphere_inertia" params="m r o_xyz o_rpy">
+    <xacro:macro name="sphere_inertia" params="m r xyz rpy">
         <inertial>
+            <origin xyz="${xyz}" rpy="${rpy}" />
             <mass value="${m}" />
-            <origin xyz="${o_xyz}" rpy="${o_rpy}" />
             <inertia ixx="${(2/5) * m * r * r}" ixy="0" ixz="0"
                      iyy="${(2/5) * m * r * r}" iyz="0"

File: src/my_robot_description/urdf/mobile_base.xacro (robot description, xacro)
@@ -21,6 +21,6 @@
             <origin xyz="0 0 ${base_height / 2.0}" rpy="0 0 0" />
         </collision>
-        <xacro:box_inertia m="5.0" x="${base_length}" y="${base_width}" z="${base_height}"
-                           o_xyz="0 0 ${base_height / 2.0}" o_rpy="0 0 0" />
+        <xacro:box_inertia m="5.0" l="${2*base_length}" w="${2*base_width}" h="${2*base_height}"
+                           xyz="0 0 ${base_height / 2.0}" rpy="0 0 0" />
     </link>
     <xacro:macro name="wheel_link" params="prefix">
@@ -35,10 +35,10 @@
             <collision>
                 <geometry>
-                    <sphere radius="${wheel_radius}" />
+                    <cylinder radius="${wheel_radius}" length="${wheel_length}" />
                 </geometry>
-                <origin xyz="0 0 0" rpy="0 0 0" />
+                <origin xyz="0 0 0" rpy="${pi / 2.0} 0 0" />
             </collision>
-            <xacro:cylinder_inertia m="1.0" r="${wheel_radius}" l="${wheel_length}"
-                                    o_xyz="0 0 0" o_rpy="${pi / 2.0} 0 0" />
+            <xacro:cylinder_inertia m="1.0" r="${2*wheel_radius}" h="${2*wheel_length}"
+                                    xyz="0 0 0" rpy="${pi / 2.0} 0 0" />
         </link>
     </xacro:macro>
@@ -59,6 +59,6 @@
             <origin xyz="0 0 0" rpy="0 0 0" />
         </collision>
-        <xacro:sphere_inertia m="0.5" r="${wheel_radius / 2.0}"
-                              o_xyz="0 0 0" o_rpy="0 0 0" />
+        <xacro:sphere_inertia m="0.5" r="${2*wheel_radius / 2.0}"
+                              xyz="0 0 0" rpy="0 0 0" />
     </link>
     <joint name="base_joint" type="fixed">

File: src/my_robot_description/urdf/mobile_base_gazebo.xacro (robot description, xacro)
@@ -1,26 +1,35 @@
 <?xml version="1.0"?>
 <robot xmlns:xacro="http://www.ros.org/wiki/xacro">
+    <gazebo reference="base_link">
+        <material>Gazebo/Blue</material>
+    </gazebo>
+    <gazebo reference="right_wheel_link">
+        <material>Gazebo/Grey</material>
+    </gazebo>
+    <gazebo reference="left_wheel_link">
+        <material>Gazebo/Grey</material>
+    </gazebo>
     <gazebo reference="caster_wheel_link">
+        <material>Gazebo/Grey</material>
         <mu1 value="0.1" />
         <mu2 value="0.1" />
     </gazebo>
     <gazebo>
-        <plugin
-            filename="gz-sim-diff-drive-system"
-            name="gz::sim::systems::DiffDrive">
+        <plugin name="diff_drive_controller" filename="libgazebo_ros_diff_drive.so">
+            <!-- Update rate in Hz -->
+            <update_rate>50</update_rate>
+            <!-- wheels -->
             <left_joint>base_left_wheel_joint</left_joint>
             <right_joint>base_right_wheel_joint</right_joint>
+            <!-- kinematics -->
             <wheel_separation>0.45</wheel_separation>
-            <wheel_radius>0.1</wheel_radius>
-            <frame_id>odom</frame_id>
-            <child_frame_id>base_footprint</child_frame_id>
-        </plugin>
-    </gazebo>
-    <gazebo>
-        <plugin
-            filename="gz-sim-joint-state-publisher-system"
-            name="gz::sim::systems::JointStatePublisher">
-            <joint_name>base_left_wheel_joint</joint_name>
-            <joint_name>base_right_wheel_joint</joint_name>
+            <wheel_diameter>0.2</wheel_diameter>
+            <!-- output -->
+            <publish_odom>true</publish_odom>
+            <publish_odom_tf>true</publish_odom_tf>
+            <publish_wheel_tf>true</publish_wheel_tf>
+            <odometry_topic>odom</odometry_topic>
+            <odometry_frame>odom</odometry_frame>
+            <robot_base_frame>base_footprint</robot_base_frame>
         </plugin>
     </gazebo>

File: src/my_robot_description/urdf/my_robot.urdf.xacro (robot description, xacro)
@@ -4,11 +4,4 @@
     <xacro:include filename="mobile_base.xacro" />
     <xacro:include filename="mobile_base_gazebo.xacro" />
-    <xacro:include filename="arm.xacro" />
-    <xacro:include filename="arm_gazebo.xacro" />
     <xacro:include filename="camera.xacro" />
-    <joint name="mobile_base_arm_joint" type="fixed">
-        <parent link="base_link" />
-        <child link="arm_base_link" />
-        <origin xyz="${base_length / 4.0} 0 ${base_height}" rpy="0 0 0" />
-    </joint>
 </robot>
